File: Hardware/SimplePlayer.kicad_pcb (KiCad board)
At the start: 6 copper layers, 0 parts

Commit message: Expander and IO
Added an IO expander to the design.
Finished the main connections between the basic components.
Parts:
- added REF**: XIAO-ESP32S3-PLUS-SMD, Custom_Parts:XIAO-ESP32S3-PLUS-SMD, F.Cu at (113.7, 86.1)
Other:
- board outline added: 60 x 40 mm
