File: Hardware/Audio.kicad_sch (KiCad schematic)
At the start: 36 parts, among them IC1 ES9039Q2M, U5 OPA1622, U6 OPA1622, U7 OPA1622, U8 OPA1622

Commit message: Expander and IO
Added an IO expander to the design.
Finished the main connections between the basic components.
Parts:
- added C31: 10n, symbol Device:C
- added R36: 22, symbol Device:R
- added Y1: 50.0MHz, Oscillator:Oscillator_SMD_Abracon_ASDMB-4Pin_2.5x2.0mm, symbol Oscillator:ASDMB-xxxMHz
- renumbered C12 to C22, C13 to C23, C14 to C24, C15 to C25, C16 to C26, C17 to C27, C18 to C28, C19 to C29, C31 to C30, C20 to C32, C32 to C33, C21 to C34, C22 to C35, C27 to C36, C28 to C37, C29 to C38, C23 to C39, C24 to C40, C30 to C41, R20 to R24, R21 to R25, R22 to R26, R23 to R27, R24 to R28, R25 to R29, R26 to R30, R27 to R31, R28 to R32, R29 to R33, R30 to R34, R31 to R35, U8 to U5
Connections:
- net 3V3D: now also C31.1, Y1.4 (VDD)
- net GND: now also C31.2, Y1.2 (GND)
- net PRE_EN: now reaches U6.8 (EN)
- net PRE_EN: now also U5.8 (EN)
- net OUT_EN: now reaches U7.8 (EN)
- net I2S_MCLK renamed MCLK
- net MCLK: now also R36.2
- new net: R36.1, Y1.3 (Out)
- no-connect marks 8 -> 9
Other:
- moved on the sheet: C22, C23, C24, C25, C26, C27, C28, C29, C30, C32, C33, C34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

Commit message: Balanced output
Updated the amplifier section, now it offers a completely balanced configuration.
Added capacitors to the audio jack for protection.
Parts:
- removed C38: 100n, symbol Device:C
- removed U5, U6: OPA1622, Package_SON:Texas_S-PVSON-N10, symbol Amplifier_Audio:OPA1622
- added C30, C31: 220p, symbol Device:C
- added C40, C42, C45: 100n, symbol Device:C
- added U5, U6: OPA1612AxD, Package_DIP:DIP-20_W7.62mm, symbol Amplifier_Operational:OPA1612AxD
- added U8: OPA1622, Package_SON:Texas_S-PVSON-N10, symbol Amplifier_Audio:OPA1622
- C22, C23, C24, C25: value 100p -> 220p
- C26, C27: value 560p -> 10p
- C28, C29: value 560p -> 220p
- R24, R25, R26, R27: value 2.32K -> 1K
- R28, R29, R30: value 1.58K -> 4.7K
- R31: value 560 -> 4.7K
- R32: value 1.58K -> 1K
- R33, R34, R35: value 560 -> 1K
- renumbered C30 to C32, C31 to C33, C33 to C34, C32 to C35, C34 to C37, C35 to C38, C37 to C39, C39 to C43, C40 to C44
Connections:
- net +4V2A: now also C40.1, C42.1, U5.8 (V+), U6.8 (V+), U8.2 (V+)
- net -4V2A: now also C45.1, U5.4 (V-), U6.4 (V-), U8.11 (V-), U8.4 (V-)
- net DAC_OUT1A: now also U5.5 (+)
- net DAC_OUT1B: now also U5.6 (-)
- net DAC_OUT2A: now also U6.5 (+)
- net DAC_OUT2B: now also U6.6 (-)
- net GND: now also C28.1, C29.1, C30.1, C31.1, C40.2, C42.2, C45.2, U5.3 (+), U6.3 (+), U8.3 (GND); no longer C26.1, C27.1, R31.1, R33.1
- net OUT_EN: now also U8.8 (EN)
- net at R33.2, U7.5 (+): now also C29.2; no longer C27.2, R29.2
- net at C23.2, R25.2: now also R29.1, R33.1, U5.7; no longer R28.1
- net at C22.2, R24.2: now also C26.2, R28.2, R32.1, U5.1; no longer R30.1
- net at R30.2, R34.1: now also C24.2, C27.2, R26.2, U6.1; no longer C28.1, U7.10 (-)
- net at C25.2, R27.2: now also R31.1, R35.1, U6.7; no longer R29.1
- removed net JACK_OUT1: C28.2, R34.2, U7.9
- removed net JACK_OUT2: C29.2, R35.2, U7.7
- new net: C26.1, R28.1, R29.2, U5.2 (-)
- new net: C27.1, R30.1, R31.2, U6.2 (-)
- new net: C31.2, R35.2, U8.5 (+)
- new net: C30.2, R34.2, U8.1 (+)
- new net: C28.2, R32.2, U7.1 (+)
- new net JACK_OUT1A: U7.10 (-), U7.9
- new net JACK_OUT1B: U7.6 (-), U7.7
- new net JACK_OUT2A: U8.10 (-), U8.9
- new net JACK_OUT2B: U8.6 (-), U8.7
Other:
- moved on the sheet: C32, C33, C34, C35, C36, C37, C38, C39, C43, C44, IC1, R36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
