File: Hardware/Expander.kicad_sch (KiCad schematic)
At the start: 27 parts, among them J5 NBA1-24-001, J6 PJ-342, SW1 SW_UP, SW2 SW_LEFT, SW3 SW_CENTER, SW4 SW_DOWN, SW5 SW_RIGHT, U8 TCA9535RTWR

Commit message: Balanced output
Updated the amplifier section, now it offers a completely balanced configuration.
Added capacitors to the audio jack for protection.
Parts:
- added C46, C47, C48, C49: 10p, symbol Device:C
- renumbered C42 to C50, C43 to C51, C44 to C52, C45 to C53, C46 to C54, J6 to J5, J5 to J6, U8 to U9
Connections:
- net JACK_OUT1 is gone; now on net JACK_OUT1A: J5.T
- net JACK_OUT2 is gone; now on net JACK_OUT2A: J5.R1
- net GND: now also J6.S (GND), C46.2, C47.2, C48.2, C49.2
- net JACK_OUT1B: now reaches J6.R1 (L-)
- net JACK_OUT1B: now also C48.1
- net JACK_OUT2A: now reaches J6.R2 (R+)
- net JACK_OUT2A: now also C47.1
- net JACK_OUT2B: now reaches J6.R3 (R-)
- net JACK_OUT2B: now also C49.1
- net JACK_OUT1A: now reaches J6.T (L+)
- net JACK_OUT1A: now also C46.1
- no-connect marks 7 -> 9
Other:
- moved on the sheet: J5, J6
