File: Hardware/Power.kicad_sch (KiCad schematic)
At the start: 23 parts, among them J3 BATTERY, J4 PJ-342, U2 TPS61040DBV, U3 TPS7A20xxxDBV, U4 LM27762

Commit message: Expander and IO
Added an IO expander to the design.
Finished the main connections between the basic components.
Parts:
- removed J4: PJ-342, Custom_Parts:JACK_3.5mm_PJ311_HOR, symbol Connector_Audio:AudioJack4_SwitchTR1
- added R18, R19: 220K, symbol Device:R
- renumbered C2 to C12, C3 to C13, C4 to C14, C5 to C15, C6 to C16, C7 to C17, C8 to C18, C9 to C19, C10 to C20, C11 to C21, D8 to D10, J3 to J4, L1 to L2, R14 to R16, R15 to R17, R16 to R20, R17 to R21, R18 to R22, R19 to R23
Connections:
- net GND: now also R19.2
- net VBAT: now also R18.1
- new net VBAT_MON: R18.2, R19.1
- no-connect marks 2 -> 0
Other:
- moved on the sheet: J4

Commit message: Balanced output
Updated the amplifier section, now it offers a completely balanced configuration.
Added capacitors to the audio jack for protection.
Parts:
- R16: value 510K -> 330K
- R17: value 200K -> 100K
- R20, R23: value 270K -> 470K
- R21, R22: value 110K -> 150K
Other:
- note added: "LM27762 regulator output voltage: 5.0V Voutp=1.2 x (R1 + R2) / R2 Voutn=-1.22 x (R3 + R4) / R4"
- note added: "TPS61040 regulator output voltage: 5.3V Vout=1.233 x (1 + R1 / R2)"
- note removed: "LM27762 regulator output voltage: 4.2V Voutp=1.2 x (R1 + R2) / R2 Voutn=-1.22 x (R3 + R4) / R4"
- note removed: "TPS61040 regulator output voltage: 4.37V Vout=1.233 x (1 + R1 / R2)"
Changed lines of the file:
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@@
 		(company "DavidMolTor")
 	)
-	(text "TPS61040 regulator output voltage: 4.37V\n\nVout=1.233 x (1 + R1 / R2)"
+	(text "TPS61040 regulator output voltage: 5.3V\n\nVout=1.233 x (1 + R1 / R2)"
 		(exclude_from_sim no)
 		(at 118.872 32.512 0)
@@
 		)
 	)
-	(text "LM27762 regulator output voltage: 4.2V\n\nVoutp=1.2 x (R1 + R2) / R2\n\nVoutn=-1.22 x (R3 + R4) / R4"
+	(text "LM27762 regulator output voltage: 5.0V\n\nVoutp=1.2 x (R1 + R2) / R2\n\nVoutn=-1.22 x (R3 + R4) / R4"
 		(exclude_from_sim no)
 		(at 195.58 34.544 0)
@@
 			)
 		)
-		(property "Value" "510K"
+		(property "Value" "330K"
 			(at 101.6 63.4999 0)
 			(show_name no)
@@
 			)
 		)
-		(property "Value" "200K"
+		(property "Value" "100K"
 			(at 101.6 76.1999 0)
 			(show_name no)
@@
 			)
 		)
-		(property "Value" "110K"
+		(property "Value" "150K"
 			(at 223.52 63.4999 0)
 			(show_name no)
@@
 			)
 		)
-		(property "Value" "270K"
+		(property "Value" "470K"
 			(at 223.52 71.1199 0)
 			(show_name no)
@@
 			)
 		)
-		(property "Value" "270K"
+		(property "Value" "470K"
 			(at 223.52 48.2599 0)
 			(show_name no)
@@
 			)
 		)
-		(property "Value" "110K"
+		(property "Value" "150K"
 			(at 223.52 55.8799 0)
 			(show_name no)
